File: Hardware/ProDOS ROM-Drive.kicad_pcb (KiCad board)
At the start: 2 copper layers, 85.7 x 54 mm, 17 parts, among them J1 Apple II Expansion Slot, U1 74LS00, U2 74LS32

Commit message: Update to KiCAD 6
Other:
- net class Default removed
- net class Ground removed
- net class Power removed

Commit message: Update schematic and fix data bus lines
Connections:
- net Net-(DataBuffer1-Pad1) renamed /~{R}/W
- net Net-(DataBuffer1-Pad19) renamed /~{IO SELECT} AND ~{DEVICE SELECT}
- net Net-(EPROM1-Pad1) renamed /CA19
- net Net-(EPROM1-Pad10) renamed /A2
- net Net-(EPROM1-Pad11) renamed /A1
- net Net-(EPROM1-Pad12) renamed /A0
- net Net-(EPROM1-Pad2) renamed /CA16
- net Net-(EPROM1-Pad22) renamed /~{ROM ENABLE}
- net Net-(EPROM1-Pad23) renamed /CA10
- net Net-(EPROM1-Pad25) renamed /CA11
- net Net-(EPROM1-Pad26) renamed /CA9
- net Net-(EPROM1-Pad27) renamed /CA8
- net Net-(EPROM1-Pad28) renamed /CA13
- net Net-(EPROM1-Pad29) renamed /CA14
- net Net-(EPROM1-Pad3) renamed /CA15
- net Net-(EPROM1-Pad30) renamed /CA17
- net Net-(EPROM1-Pad31) renamed /CA18
- net Net-(EPROM1-Pad4) renamed /CA12
- net Net-(EPROM1-Pad5) renamed /CA7
- net Net-(EPROM1-Pad6) renamed /CA6
- net Net-(EPROM1-Pad7) renamed /CA5
- net Net-(EPROM1-Pad8) renamed /CA4
- net Net-(EPROM1-Pad9) renamed /A3
- net Net-(HiAddrBuffer1-Pad19) renamed /~{IO SELECT}
- net Net-(HiAddrLatch1-Pad1) renamed /~{DEVICE SELECT}
- net Net-(HiAddrLatch1-Pad11) renamed /~{HIGH LATCH ENABLE}
- net Net-(J1-Pad18) renamed /R/~{W}
- net Net-(J1-Pad23) renamed /INT
- net Net-(J1-Pad24) renamed /DMA
- net Net-(J1-Pad6) renamed /A4
- net Net-(J1-Pad7) renamed /A5
- net Net-(J1-Pad8) renamed /A6
- net Net-(J1-Pad9) renamed /A7
- net Net-(LowAddrLatch1-Pad11) renamed /~{LOW LATCH ENABLE}
- net Net-(U1-Pad11) renamed /~{A0}
- DataBuffer1 pad 11: Net-(DataBuffer1-Pad11) -> /CD7
- DataBuffer1 pad 12: Net-(DataBuffer1-Pad12) -> /CD6
- DataBuffer1 pad 13: Net-(DataBuffer1-Pad13) -> /CD5
- DataBuffer1 pad 14: Net-(DataBuffer1-Pad14) -> /CD4
- DataBuffer1 pad 15: Net-(DataBuffer1-Pad15) -> /CD3
- DataBuffer1 pad 16: Net-(DataBuffer1-Pad16) -> /CD2
- DataBuffer1 pad 17: Net-(DataBuffer1-Pad17) -> /CD1
- DataBuffer1 pad 18: Net-(DataBuffer1-Pad18) -> /CD0
- DataBuffer1 pad 2: Net-(DataBuffer1-Pad2) -> /D0
- DataBuffer1 pad 3: Net-(DataBuffer1-Pad3) -> /D1
- DataBuffer1 pad 4: Net-(DataBuffer1-Pad4) -> /D2
- DataBuffer1 pad 5: Net-(DataBuffer1-Pad5) -> /D3
- DataBuffer1 pad 6: Net-(DataBuffer1-Pad6) -> /D4
- DataBuffer1 pad 7: Net-(DataBuffer1-Pad7) -> /D5
- DataBuffer1 pad 8: Net-(DataBuffer1-Pad8) -> /D6
- DataBuffer1 pad 9: Net-(DataBuffer1-Pad9) -> /D7
- EPROM1 pad 13: Net-(DataBuffer1-Pad18) -> /CD0
- EPROM1 pad 14: Net-(DataBuffer1-Pad17) -> /CD1
- EPROM1 pad 15: Net-(DataBuffer1-Pad16) -> /CD2
- EPROM1 pad 17: Net-(DataBuffer1-Pad15) -> /CD3
- EPROM1 pad 18: Net-(DataBuffer1-Pad14) -> /CD4
- EPROM1 pad 19: Net-(DataBuffer1-Pad13) -> /CD5
- EPROM1 pad 20: Net-(DataBuffer1-Pad12) -> /CD6
- EPROM1 pad 21: Net-(DataBuffer1-Pad11) -> /CD7
- HiAddrLatch1 pad 13: Net-(DataBuffer1-Pad6) -> /CD4
- HiAddrLatch1 pad 14: Net-(DataBuffer1-Pad7) -> /CD5
- HiAddrLatch1 pad 17: Net-(DataBuffer1-Pad8) -> /CD6
- HiAddrLatch1 pad 18: Net-(DataBuffer1-Pad9) -> /CD7
- HiAddrLatch1 pad 3: Net-(DataBuffer1-Pad2) -> /CD0
- HiAddrLatch1 pad 4: Net-(DataBuffer1-Pad3) -> /CD1
- HiAddrLatch1 pad 7: Net-(DataBuffer1-Pad4) -> /CD2
- HiAddrLatch1 pad 8: Net-(DataBuffer1-Pad5) -> /CD3
- J1 pad 10: (no net) -> unconnected-(J1-Pad10)
- J1 pad 11: (no net) -> unconnected-(J1-Pad11)
- J1 pad 12: (no net) -> unconnected-(J1-Pad12)
- J1 pad 13: (no net) -> unconnected-(J1-Pad13)
- J1 pad 14: (no net) -> unconnected-(J1-Pad14)
- J1 pad 15: (no net) -> unconnected-(J1-Pad15)
- J1 pad 16: (no net) -> unconnected-(J1-Pad16)
- J1 pad 17: (no net) -> unconnected-(J1-Pad17)
- J1 pad 19: (no net) -> unconnected-(J1-Pad19)
- J1 pad 20: (no net) -> unconnected-(J1-Pad20)
- J1 pad 21: (no net) -> unconnected-(J1-Pad21)
- J1 pad 22: (no net) -> unconnected-(J1-Pad22)
- J1 pad 29: (no net) -> unconnected-(J1-Pad29)
- J1 pad 30: (no net) -> unconnected-(J1-Pad30)
- J1 pad 31: (no net) -> unconnected-(J1-Pad31)
- J1 pad 32: (no net) -> unconnected-(J1-Pad32)
- J1 pad 33: (no net) -> unconnected-(J1-Pad33)
- J1 pad 34: (no net) -> unconnected-(J1-Pad34)
- J1 pad 35: (no net) -> unconnected-(J1-Pad35)
- J1 pad 36: (no net) -> unconnected-(J1-Pad36)
- J1 pad 37: (no net) -> unconnected-(J1-Pad37)
- J1 pad 38: (no net) -> unconnected-(J1-Pad38)
- J1 pad 39: (no net) -> unconnected-(J1-Pad39)
- J1 pad 40: (no net) -> unconnected-(J1-Pad40)
- J1 pad 42: Net-(DataBuffer1-Pad9) -> /D7
- J1 pad 43: Net-(DataBuffer1-Pad8) -> /D6
- J1 pad 44: Net-(DataBuffer1-Pad7) -> /D5
- J1 pad 45: Net-(DataBuffer1-Pad6) -> /D4
- J1 pad 46: Net-(DataBuffer1-Pad5) -> /D3
- J1 pad 47: Net-(DataBuffer1-Pad4) -> /D2
- J1 pad 48: Net-(DataBuffer1-Pad3) -> /D1
- J1 pad 49: Net-(DataBuffer1-Pad2) -> /D0
- J1 pad 50: (no net) -> unconnected-(J1-Pad50)
- LowAddrLatch1 pad 13: Net-(DataBuffer1-Pad6) -> /CD4
- LowAddrLatch1 pad 14: Net-(DataBuffer1-Pad7) -> /CD5
- LowAddrLatch1 pad 17: Net-(DataBuffer1-Pad8) -> /CD6
- LowAddrLatch1 pad 18: Net-(DataBuffer1-Pad9) -> /CD7
- LowAddrLatch1 pad 3: Net-(DataBuffer1-Pad2) -> /CD0
- LowAddrLatch1 pad 4: Net-(DataBuffer1-Pad3) -> /CD1
- LowAddrLatch1 pad 7: Net-(DataBuffer1-Pad4) -> /CD2
- LowAddrLatch1 pad 8: Net-(DataBuffer1-Pad5) -> /CD3
Routing:
- net /CD1: track 0.00 -> 80.7 mm, vias 0 -> 2
- net /CD6: track 0.00 -> 79.8 mm, vias 0 -> 1
- net /CD5: track 0.00 -> 75.1 mm, vias 0 -> 1
- net /CD7: track 0.00 -> 74.9 mm
- net /CD0: track 0.00 -> 73.3 mm, vias 0 -> 1
- net /CD2: track 0.00 -> 70.0 mm
- net Net-(DataBuffer1-Pad9): track 67.7 -> 0.00 mm
- net /CD4: track 0.00 -> 61.6 mm, vias 0 -> 1
- net /CD3: track 0.00 -> 61.0 mm, vias 0 -> 1
- net Net-(DataBuffer1-Pad8): track 60.7 -> 0.00 mm
- net Net-(DataBuffer1-Pad2): track 59.8 -> 0.00 mm, vias 1 -> 0
- net Net-(DataBuffer1-Pad3): track 57.2 -> 0.00 mm, vias 1 -> 0
- net Net-(DataBuffer1-Pad7): track 52.9 -> 0.00 mm, vias 1 -> 0
- net Net-(DataBuffer1-Pad4): track 51.1 -> 0.00 mm
- net Net-(DataBuffer1-Pad6): track 49.3 -> 0.00 mm, vias 1 -> 0
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Other:
- board text added: "ProDOS ROM-Drive v4.0 (c)1998-2022 Terence J. Boldt https://github.com/tjboldt/ProDOS-ROM-Drive"
- board text added: "ProDOS ROM-Drive v4.0 For Apple ][ computers Bootable 1 MB read-only solid state disk (c)1998-2022 Terence J. Boldt https://github.com/tjboldt/ProDOS-ROM-Drive"
- board text removed: "ProDOS ROM-Drive v3.0 (c)1998-2021 Terence J. Boldt https://github.com/tjboldt/ProDOS-ROM-Drive"
- board text removed: "ProDOS ROM-Drive v3.0 For Apple ][ computers Bootable 1 MB read-only solid state disk (c)1998-2021 Terence J. Boldt https://github.com/tjboldt/ProDOS-ROM-Drive"
